File: hardware/panel-art/panel-art.kicad_pcb (KiCad board)
At the start: 2 copper layers, 0 parts

Commit message: Added board layout page.
Other:
- board text added: "AN"
- board text removed: "AUTO NOTCH"
- board text removed: "PWR"
