File: hardware/audio filter.kicad_pcb (KiCad board)
At the start: 2 copper layers, 0 parts

Commit message: Revision A (Prototype).
Other:
- board outline added: 100 x 75 mm
- board text removed: "ALE in"
- board text removed: "Audio in"
- board text removed: "Auto Notch"
- board text removed: "Ch. Filter in"
- board text removed: "DASH"
- board text removed: "DBG1"
- board text removed: "DBG2"
- board text removed: "DOT"
- board text removed: "FILTER MODE"
- board text removed: "GND"
- board text removed: "GPIO12"
- board text removed: "GPIO13"
- board text removed: "GPIO3"
- board text removed: "Ground to activate"
- board text removed: "Height restriction is 15mm above PCB level."
- board text removed: "KEY IN"
- board text removed: "KEY OUT"
- board text removed: "Key out"
- board text removed: "NC"
- board text removed: "Spkr En (to GND to enable)"
- board text removed: "Spkr audio in"
- board text removed: "Spkr audio out"
- board text removed: "TUNE"
